File: src/hw/TOSMETRE18F1320/TOSMETRE18F1320.kicad_pcb (KiCad board)
At the start: 2 copper layers, 13 parts, among them J1 Conn_01x01_Female, J2 Conn_01x01_Female, J3 REF, J4 FWD, U1 L7805, Y1 Crystal

Commit message: realisation rapide PCD 18f1320 a optimiser
Parts:
- added U2: 18F1320_SSOP, SMD_Packages:SSOP-20, F.Cu at (203.2, 109.2)
- moved Y1 138.3 mm to (213.4, 116.8)
- moved C5 128.5 mm to (219.5, 111.8), turned to 180 degrees
- moved C4 121.1 mm to (211.9, 111.8)
- moved J3 120.1 mm to (215.9, 109.2)
- moved C2 90.5 mm to (181.4, 114.3), turned to 180 degrees
- moved J4 88.7 mm to (215.9, 104.1)
- moved C1 82.0 mm to (172.7, 113.3), turned to 270 degrees
- moved D1 76.5 mm to (167.6, 103.1), turned to 90 degrees
- moved J2 68.9 mm to (167.6, 109.2)
- moved U1 45.5 mm to (172.7, 108.1)
- moved C3 35.9 mm to (194.1, 111.8)
- moved J1 35.8 mm to (167.6, 96.5)
Routing:
- net Net-(DS1-Pad4): track 0.00 -> 51.8 mm
- net Net-(DS1-Pad6): track 0.00 -> 43.2 mm
- net GNDREF: track 0.00 -> 34.8 mm, vias 0 -> 5
- net Net-(C2-Pad1): track 0.00 -> 30.6 mm
- net Net-(C5-Pad2): track 0.00 -> 21.8 mm
- net Net-(C4-Pad2): track 0.00 -> 15.9 mm
- net Net-(J3-Pad1): track 0.00 -> 12.9 mm
- net Net-(J4-Pad1): track 0.00 -> 12.3 mm
- net Net-(DS1-Pad14): track 0.00 -> 12.3 mm
- net Net-(DS1-Pad13): track 0.00 -> 11.2 mm
- net Net-(C1-Pad1): track 0.00 -> 10.9 mm
- net Net-(DS1-Pad12): track 0.00 -> 10.5 mm
- net Net-(DS1-Pad11): track 0.00 -> 10.5 mm
- net Net-(C3-Pad2): track 0.00 -> 9.19 mm
- net Net-(D1-Pad2): track 0.00 -> 5.08 mm
- added copper zone on B.Cu, net GNDREF
