File: src/hw/TOSMETRE18F1320/TOSMETRE18F1320.sch (KiCad schematic (older format))
At the start: 14 parts, among them J1 Conn_01x01_Female, J2 Conn_01x01_Female, J3 REF, J4 FWD, U1 L7805, U2 18F1320_SSOP, Y1 Crystal

Commit message: realisation rapide PCD 18f1320 a optimiser
Parts:
- U2: footprint (none) -> SMD_Packages:SSOP-20
Changed lines of the file:
@@
 $EndComp
 $Comp
-L GNDREF #PWR7
+L GNDREF #PWR01
 U 1 1 5AB2782F
 P 7750 3550
-F 0 "#PWR7" H 7750 3300 50  0001 C CNN
+F 0 "#PWR01" H 7750 3300 50  0001 C CNN
 F 1 "GNDREF" H 7750 3400 50  0000 C CNN
 F 2 "" H 7750 3550 50  0001 C CNN
@@
 $EndComp
 $Comp
-L GNDREF #PWR10
+L GNDREF #PWR02
 U 1 1 5AB27830
 P 9400 1950
-F 0 "#PWR10" H 9400 1700 50  0001 C CNN
+F 0 "#PWR02" H 9400 1700 50  0001 C CNN
 F 1 "GNDREF" H 9400 1800 50  0000 C CNN
 F 2 "" H 9400 1950 50  0001 C CNN
@@
 $EndComp
 $Comp
-L GNDREF #PWR9
+L GNDREF #PWR03
 U 1 1 5AB27833
 P 8450 6050
-F 0 "#PWR9" H 8450 5800 50  0001 C CNN
+F 0 "#PWR03" H 8450 5800 50  0001 C CNN
 F 1 "GNDREF" H 8450 5900 50  0000 C CNN
 F 2 "" H 8450 6050 50  0001 C CNN
@@
 $EndComp
 $Comp
-L GNDREF #PWR8
+L GNDREF #PWR04
 U 1 1 5AB27834
 P 8200 3550
-F 0 "#PWR8" H 8200 3300 50  0001 C CNN
+F 0 "#PWR04" H 8200 3300 50  0001 C CNN
 F 1 "GNDREF" H 8200 3400 50  0000 C CNN
 F 2 "" H 8200 3550 50  0001 C CNN
@@
 $EndComp
 $Comp
-L GNDREF #PWR5
+L GNDREF #PWR05
 U 1 1 5AB27835
 P 5400 2450
-F 0 "#PWR5" H 5400 2200 50  0001 C CNN
+F 0 "#PWR05" H 5400 2200 50  0001 C CNN
 F 1 "GNDREF" H 5400 2300 50  0000 C CNN
 F 2 "" H 5400 2450 50  0001 C CNN
@@
 $EndComp
 $Comp
-L GNDREF #PWR3
+L GNDREF #PWR06
 U 1 1 5AB27836
 P 4800 2450
-F 0 "#PWR3" H 4800 2200 50  0001 C CNN
+F 0 "#PWR06" H 4800 2200 50  0001 C CNN
 F 1 "GNDREF" H 4800 2300 50  0000 C CNN
 F 2 "" H 4800 2450 50  0001 C CNN
@@
 $EndComp
 $Comp
-L GNDREF #PWR4
+L GNDREF #PWR07
 U 1 1 5AB27837
 P 4800 2450
-F 0 "#PWR4" H 4800 2200 50  0001 C CNN
+F 0 "#PWR07" H 4800 2200 50  0001 C CNN
 F 1 "GNDREF" H 4800 2300 50  0000 C CNN
 F 2 "" H 4800 2450 50  0001 C CNN
@@
 $EndComp
 $Comp
-L GNDREF #PWR1
+L GNDREF #PWR08
 U 1 1 5AB2783B
 P 3900 2450
-F 0 "#PWR1" H 3900 2200 50  0001 C CNN
+F 0 "#PWR08" H 3900 2200 50  0001 C CNN
 F 1 "GNDREF" H 3900 2300 50  0000 C CNN
 F 2 "" H 3900 2450 50  0001 C CNN
@@
 $EndComp
 $Comp
-L GNDREF #PWR2
+L GNDREF #PWR09
 U 1 1 5AB2783C
 P 3900 2450
-F 0 "#PWR2" H 3900 2200 50  0001 C CNN
+F 0 "#PWR09" H 3900 2200 50  0001 C CNN
 F 1 "GNDREF" H 3900 2300 50  0000 C CNN
 F 2 "" H 3900 2450 50  0001 C CNN
@@
 $EndComp
 $Comp
-L GNDREF #PWR6
+L GNDREF #PWR010
 U 1 1 5AB27842
 P 5900 2450
-F 0 "#PWR6" H 5900 2200 50  0001 C CNN
+F 0 "#PWR010" H 5900 2200 50  0001 C CNN
 F 1 "GNDREF" H 5900 2300 50  0000 C CNN
 F 2 "" H 5900 2450 50  0001 C CNN
@@
 F 0 "U2" H 8350 5925 50  0000 R CNN
 F 1 "18F1320_SSOP" H 8550 6000 50  0000 R CNN
-F 2 "" H 7000 5050 50  0001 L CNN
+F 2 "SMD_Packages:SSOP-20" H 7000 5050 50  0001 L CNN
 F 3 "" H 8250 4750 50  0001 C CNN
 	1    8450 5350
